File: Comutator.sch (KiCad schematic (older format))
At the start: 19 parts, among them J1 Conn_01x02, J2 Conn_01x02, K1 FINDER-40.52, Q1 IRLML2402, Q2 IRLML2402, Q3 BT139-600, U1 MOC3063M

Commit message: Add input connector
Parts:
- removed J1: Conn_01x02, symbol Connector_Generic:Conn_01x02
- added J1: Conn_01x03, symbol Connector_Generic:Conn_01x03
Connections:
- wire segments 81 -> 83
Changed lines of the file:
@@
 EESchema Schematic File Version 4
+LIBS:Comutator-cache
 EELAYER 26 0
 EELAYER END
@@
 	8900 4650 8750 4650
 Connection ~ 8050 4650
-$Comp
-L Connector_Generic:Conn_01x02 J1
-U 1 1 5B23FE1D
-P 3600 4250
-F 0 "J1" H 3520 4467 50  0000 C CNN
-F 1 "Conn_01x02" H 3520 4376 50  0000 C CNN
-F 2 "" H 3600 4250 50  0001 C CNN
-F 3 "~" H 3600 4250 50  0001 C CNN
-	1    3600 4250
-	-1   0    0    -1
-$EndComp
 Wire Wire Line
 	3800 4250 4100 4250
@@
 Wire Wire Line
 	8750 4650 8050 4650
+$Comp
+L Connector_Generic:Conn_01x03 J1
+U 1 1 5B253C52
+P 3600 4250
+F 0 "J1" H 3520 4567 50  0000 C CNN
+F 1 "Conn_01x03" H 3520 4476 50  0000 C CNN
+F 2 "" H 3600 4250 50  0001 C CNN
+F 3 "~" H 3600 4250 50  0001 C CNN
+	1    3600 4250
+	-1   0    0    -1
+$EndComp
+$Comp
+L power:+5V #PWR04
+U 1 1 5B253CE5
+P 4000 4000
+F 0 "#PWR04" H 4000 3850 50  0001 C CNN
+F 1 "+5V" H 4015 4173 50  0000 C CNN
+F 2 "" H 4000 4000 50  0001 C CNN
+F 3 "" H 4000 4000 50  0001 C CNN
+	1    4000 4000
+	1    0    0    -1
+$EndComp
+Wire Wire Line
+	4000 4000 4000 4150
+Wire Wire Line
+	4000 4150 3800 4150
 $EndSCHEMATC

Commit message: Add SO-6 package
Parts:
- U1: footprint (none) -> comutator:SO-6
Changed lines of the file:
@@
 F 0 "U1" H 6900 4675 50  0000 C CNN
 F 1 "MOC3063M" H 6900 4584 50  0000 C CNN
-F 2 "" H 6700 4150 50  0001 L CIN
+F 2 "comutator:SO-6" H 6700 4150 50  0001 L CIN
 F 3 "http://www.fairchildsemi.com/ds/MO/MOC3061M.pdf" H 6865 4350 50  0001 L CNN
 	1    6900 4350

Commit message: Create pcb
Parts:
- C1, C2: footprint Capacitor_SMD:C_1206_3216Metric -> Capacitor_SMD:C_0805_2012Metric
- D2: footprint (none) -> Diode_SMD:D_MiniMELF
- D3: footprint (none) -> LED_THT:LED_D3.0mm
- J1: footprint (none) -> Connector_PinHeader_2.54mm:PinHeader_1x03_P2.54mm_Vertical
- R1, R2, R3, R4, R5: footprint Resistor_SMD:R_0603_1608Metric -> Resistor_SMD:R_0805_2012Metric
- U1: footprint comutator:SO-6 -> Package_DIP:DIP-6_W7.62mm
Changed lines of the file:
@@
 F 0 "U1" H 6900 4675 50  0000 C CNN
 F 1 "MOC3063M" H 6900 4584 50  0000 C CNN
-F 2 "comutator:SO-6" H 6700 4150 50  0001 L CIN
+F 2 "Package_DIP:DIP-6_W7.62mm" H 6700 4150 50  0001 L CIN
 F 3 "http://www.fairchildsemi.com/ds/MO/MOC3061M.pdf" H 6865 4350 50  0001 L CNN
 	1    6900 4350
@@
 F 0 "R4" V 5643 2450 50  0000 C CNN
 F 1 "1k" V 5734 2450 50  0000 C CNN
-F 2 "Resistor_SMD:R_0603_1608Metric" V 5780 2450 50  0001 C CNN
+F 2 "Resistor_SMD:R_0805_2012Metric" V 5780 2450 50  0001 C CNN
 F 3 "~" H 5850 2450 50  0001 C CNN
 	1    5850 2450
@@
 F 0 "D3" H 6191 2666 50  0000 C CNN
 F 1 "LED" H 6191 2575 50  0000 C CNN
-F 2 "" H 6200 2450 50  0001 C CNN
+F 2 "LED_THT:LED_D3.0mm" H 6200 2450 50  0001 C CNN
 F 3 "~" H 6200 2450 50  0001 C CNN
 	1    6200 2450
@@
 F 0 "D2" H 5950 2576 50  0000 C CNN
 F 1 "BZG05C9V1" H 5950 2485 50  0000 C CNN
-F 2 "" H 5950 2700 50  0001 C CNN
+F 2 "Diode_SMD:D_MiniMELF" H 5950 2700 50  0001 C CNN
 F 3 "~" H 5950 2700 50  0001 C CNN
 	1    5950 2700
@@
 F 0 "R5" H 6520 3596 50  0000 L CNN
 F 1 "510" H 6520 3505 50  0000 L CNN
-F 2 "Resistor_SMD:R_0603_1608Metric" V 6380 3550 50  0001 C CNN
+F 2 "Resistor_SMD:R_0805_2012Metric" V 6380 3550 50  0001 C CNN
 F 3 "~" H 6450 3550 50  0001 C CNN
 	1    6450 3550
@@
 F 0 "R2" V 4593 3600 50  0000 C CNN
 F 1 "100k" V 4684 3600 50  0000 C CNN
-F 2 "Resistor_SMD:R_0603_1608Metric" V 4730 3600 50  0001 C CNN
+F 2 "Resistor_SMD:R_0805_2012Metric" V 4730 3600 50  0001 C CNN
 F 3 "~" H 4800 3600 50  0001 C CNN
 	1    4800 3600
@@
 F 0 "R3" V 4593 4850 50  0000 C CNN
 F 1 "100k" V 4684 4850 50  0000 C CNN
-F 2 "Resistor_SMD:R_0603_1608Metric" V 4730 4850 50  0001 C CNN
+F 2 "Resistor_SMD:R_0805_2012Metric" V 4730 4850 50  0001 C CNN
 F 3 "~" H 4800 4850 50  0001 C CNN
 	1    4800 4850
@@
 F 0 "R1" V 4043 4250 50  0000 C CNN
 F 1 "1k" V 4134 4250 50  0000 C CNN
-F 2 "Resistor_SMD:R_0603_1608Metric" V 4180 4250 50  0001 C CNN
+F 2 "Resistor_SMD:R_0805_2012Metric" V 4180 4250 50  0001 C CNN
 F 3 "~" H 4250 4250 50  0001 C CNN
 	1    4250 4250
@@
 F 0 "C1" H 5365 3896 50  0000 L CNN
 F 1 "1u" H 5365 3805 50  0000 L CNN
-F 2 "Capacitor_SMD:C_1206_3216Metric" H 5288 3700 50  0001 C CNN
+F 2 "Capacitor_SMD:C_0805_2012Metric" H 5288 3700 50  0001 C CNN
 F 3 "~" H 5250 3850 50  0001 C CNN
 	1    5250 3850
@@
 F 0 "C2" H 5365 5146 50  0000 L CNN
 F 1 "1u" H 5365 5055 50  0000 L CNN
-F 2 "Capacitor_SMD:C_1206_3216Metric" H 5288 4950 50  0001 C CNN
+F 2 "Capacitor_SMD:C_0805_2012Metric" H 5288 4950 50  0001 C CNN
 F 3 "~" H 5250 5100 50  0001 C CNN
 	1    5250 5100
@@
 L Connector_Generic:Conn_01x02 J2
 U 1 1 5B23E3AC
-P 9250 4250
-F 0 "J2" H 9330 4242 50  0000 L CNN
-F 1 "Conn_01x02" H 9330 4151 50  0000 L CNN
-F 2 "w_conn_screw:mors_2p" H 9250 4250 50  0001 C CNN
-F 3 "~" H 9250 4250 50  0001 C CNN
-	1    9250 4250
-	1    0    0    -1
+P 9250 4350
+F 0 "J2" H 9330 4342 50  0000 L CNN
+F 1 "Conn_01x02" H 9330 4251 50  0000 L CNN
+F 2 "w_conn_screw:mors_2p" H 9250 4350 50  0001 C CNN
+F 3 "~" H 9250 4350 50  0001 C CNN
+	1    9250 4350
+	1    0    0    1
 $EndComp
 Wire Wire Line
@@
 F 0 "J1" H 3520 4567 50  0000 C CNN
 F 1 "Conn_01x03" H 3520 4476 50  0000 C CNN
-F 2 "" H 3600 4250 50  0001 C CNN
+F 2 "Connector_PinHeader_2.54mm:PinHeader_1x03_P2.54mm_Vertical" H 3600 4250 50  0001 C CNN
 F 3 "~" H 3600 4250 50  0001 C CNN
 	1    3600 4250
